File: KiCad/ColorMemo/ColorMemo.kicad_pcb (KiCad board)
At the start: 2 copper layers, 49 parts, among them SW1 SW_Push, SW10 SW_Push, SW11 SW_Push, SW12 SW_Push, SW13 SW_Push, SW14 SW_Push, SW15 SW_Push, SW16 SW_Push, SW17 SW_Push, SW18 SW_Push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

Commit message: added kicad project
Signed-off-by: Michal Pelka <michalpelka@gmail.com>
Parts:
- SW1, SW10, SW11, SW12, SW13, SW14, SW15, SW16, SW17, SW18, SW19, SW2, SW20, SW21, SW22, SW23, SW24, SW3, SW4, SW5, SW6, SW7, SW8, SW9: footprint Button_Switch_THT:SW_PUSH-12mm -> Button_Switch_THT:SW_PUSH_6mm
- U1: moved to B.Cu
- moved U1 178.1 mm to (202.8, 70.4)
- moved D4 130.4 mm to (234.8, 44.0), turned to 180 degrees
- moved SW18 129.0 mm to (101.0, 122.5)
- moved SW17 128.2 mm to (101.0, 104.0)
- moved D12 109.1 mm to (235.2, 114.7), turned to 180 degrees
- moved SW10 108.4 mm to (101.2, 86.5)
- moved SW9 108.0 mm to (101.2, 67.8)
- moved SW3 107.4 mm to (188.2, 31.8)
- moved C9 106.9 mm to (96.2, 116.8), turned to 90 degrees
- moved D5 104.7 mm to (235.2, 79.7), turned to 180 degrees
- moved SW5 97.6 mm to (107.2, 56.2), turned to 180 degrees
- moved C12 97.2 mm to (226.8, 113.7), turned to 90 degrees
- moved SW22 96.2 mm to (188.5, 122.0)
- moved D3 94.8 mm to (190.8, 44.0), turned to 180 degrees
- moved SW2 89.8 mm to (145.0, 32.0)
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Connections:
- D10 pad 1: GND -> VCC
- D10 pad 3: VCC -> GND
- D11 pad 4: Net-(D10-DIN) -> Net-(D10-DOUT)
- D2 pad 1: GND -> VCC
- D2 pad 2: Net-(D1-DOUT) -> Net-(D2-DOUT)
- D2 pad 3: VCC -> GND
- D2 pad 4: Net-(D2-DIN) -> Net-(D1-DOUT)
- D3 pad 4: Net-(D2-DIN) -> Net-(D2-DOUT)
- D6 pad 1: GND -> VCC
- D6 pad 2: Net-(D5-DOUT) -> Net-(D6-DOUT)
- D6 pad 3: VCC -> GND
- D6 pad 4: Net-(D6-DIN) -> Net-(D5-DOUT)
- D7 pad 4: Net-(D6-DIN) -> Net-(D6-DOUT)
- D8 pad 2: unconnected-(D8-DOUT-Pad2) -> Net-(D8-DOUT)
- D9 pad 2: Net-(D10-DOUT) -> Net-(D10-DIN)
- D9 pad 4: unconnected-(D9-DIN-Pad4) -> Net-(D8-DOUT)
- SW17 pad 2: /MUL_ROW_1 -> /MUL_ROW_2
- SW18 pad 2: /MUL_ROW_1 -> /MUL_ROW_2
- SW19 pad 2: /MUL_ROW_1 -> /MUL_ROW_2
- SW20 pad 2: /MUL_ROW_1 -> /MUL_ROW_2
- SW21 pad 2: /MUL_ROW_1 -> /MUL_ROW_2
- SW22 pad 2: /MUL_ROW_1 -> /MUL_ROW_2
- SW23 pad 2: /MUL_ROW_1 -> /MUL_ROW_2
- SW24 pad 2: /MUL_ROW_1 -> /MUL_ROW_2
Routing:
- net GND: track 0.00 -> 572.8 mm, vias 0 -> 4
- net VCC: track 0.00 -> 549.0 mm, vias 0 -> 4
- net /MUL_ROW_2: track 0.00 -> 377.8 mm
- net /MUL_ROW_0: track 0.00 -> 313.5 mm
- net /MUL_ROW_1: track 0.00 -> 310.8 mm
- net /MUL_COL_0: track 0.00 -> 275.3 mm
- net /MUL_COL_3: track 0.00 -> 198.2 mm
- net /MUL_COL_1: track 0.00 -> 192.1 mm
- net Net-(D1-DIN): track 0.00 -> 186.9 mm, vias 0 -> 1
- net /MUL_COL_2: track 0.00 -> 153.1 mm
- net Net-(D5-DOUT): track 0.00 -> 58.6 mm
- net Net-(D4-DOUT): track 0.00 -> 55.0 mm, vias 0 -> 2
- net Net-(D8-DOUT): track 0.00 -> 51.4 mm, vias 0 -> 2
- net Net-(D7-DOUT): track 0.00 -> 51.1 mm
- net Net-(D6-DOUT): track 0.00 -> 50.9 mm
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Other:
- board outline added: 160.8 x 105.5 mm

Commit message: order to jlcpcb
Signed-off-by: Michal Pelka <michalpelka@gmail.com>
Parts:
- added BZ1: Buzzer, Buzzer_Beeper:Buzzer_12x9.5RM7.6, B.Cu at (128.0, 64.0)
- added C13: C_Polarized, Capacitor_THT:CP_Radial_D8.0mm_P5.00mm, B.Cu at (115.6, 64.6)
- added D13: 1N4148WT, Diode_SMD:D_SOD-523, F.Cu at (179.7, 49.8)
- added H1: MountingHole, MountingHole:MountingHole_3.2mm_M3, F.Cu at (50.0, 148.0)
- added H2: MountingHole, MountingHole:MountingHole_3.2mm_M3, F.Cu at (50.0, 50.0)
- added H3: MountingHole, MountingHole:MountingHole_3.2mm_M3, F.Cu at (204.0, 50.0)
- added H4: MountingHole, MountingHole:MountingHole_3.2mm_M3, F.Cu at (204.0, 148.0)
- added H5: MountingHole, MountingHole:MountingHole_3.2mm_M3, F.Cu at (127.0, 99.0)
- added H6: MountingHole, MountingHole:MountingHole_3.2mm_M3, F.Cu at (127.0, 148.2)
- added H7: MountingHole, MountingHole:MountingHole_3.2mm_M3, F.Cu at (3.48, 3.48)
- added H8: MountingHole, MountingHole:MountingHole_3.2mm_M3, F.Cu at (127.0, 50.0)
- added J1: Conn_01x02, Connector_JST:JST_PH_B2B-PH-K_1x02_P2.00mm_Vertical, B.Cu at (52.0, 90.0)
- added Q1: MMFTN3402, Package_TO_SOT_SMD:SOT-23, F.Cu at (179.2, 53.4)
- added R1: R100, Resistor_SMD:R_0805_2012Metric_Pad1.20x1.40mm_HandSolder, F.Cu at (167.2, 80.6)
- added R2: 100k, Resistor_SMD:R_0805_2012Metric_Pad1.20x1.40mm_HandSolder, F.Cu at (167.2, 76.4)
- added R3: R330, Resistor_SMD:R_0805_2012Metric_Pad1.20x1.40mm_HandSolder, F.Cu at (167.2, 85.6)
- moved C11 47.9 mm to (141.8, 136.3)
- moved C12 47.9 mm to (184.1, 135.5)
- moved D11 47.9 mm to (149.4, 136.9)
- moved SW20 47.9 mm to (102.3, 143.8)
- moved SW22 47.9 mm to (145.8, 143.8)
- moved SW24 47.9 mm to (189.3, 143.8)
- moved C2 47.9 mm to (97.8, 66.5)
- moved C3 47.9 mm to (142.8, 66.6)
- moved C4 47.9 mm to (199.1, 61.6)
- moved C5 47.9 mm to (188.1, 100.6)
- moved C6 47.9 mm to (141.1, 99.3)
- moved C7 47.9 mm to (98.3, 100.4)
- moved C8 47.9 mm to (52.1, 101.5)
- moved D2 47.9 mm to (104.9, 65.8)
- moved D3 47.9 mm to (148.1, 65.8)
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Connections:
- U1 pad 13: unconnected-(U1-SDA/D2-Pad13) -> Net-(U1-SDA/D2)
- U1 pad 14: Net-(D1-DIN) -> Net-(U1-SCL/D1)
Routing:
- net VCC: track 549.0 -> 609.7 mm, vias 4 -> 5
- net GND: track 572.8 -> 632.1 mm
- net Net-(BZ1--): track 0.00 -> 54.9 mm
- net Net-(D1-DIN): track 186.9 -> 224.1 mm, vias 1 -> 2
- net Net-(Q1-G): track 0.00 -> 36.2 mm, vias 0 -> 2
- net /MUL_COL_0: track 275.3 -> 293.0 mm
- net Net-(U1-SDA/D2): track 0.00 -> 16.8 mm
- net Net-(U1-SCL/D1): track 0.00 -> 15.4 mm
- net /MUL_ROW_2: track 377.8 -> 379.1 mm
- net Net-(D6-DOUT): track 50.9 -> 52.0 mm
- net /MUL_ROW_1: track 310.8 -> 311.6 mm

Commit message: Added readme, CAD
Signed-off-by: Michal Pelka <michalpelka@gmail.com>
Parts:
- added R4: 10k, Resistor_SMD:R_0805_2012Metric_Pad1.20x1.40mm_HandSolder, F.Cu at (167.0, 89.2)
Routing:
- net VDD: track 0.00 -> 19.2 mm
- net /MUL_COL_3: track 198.2 -> 206.0 mm
Changed lines of the file:
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@@
 		(tenting front back)
 		(pcbplotparams
-			(layerselection 0x00000000_00000000_55555555_5755f5ff)
+			(layerselection 0x00000000_00000000_55555555_57555550)
 			(plot_on_all_layers_selection 0x00000000_00000000_00000000_00000000)
 			(disableapertmacros no)
@@
 			(plotframeref no)
 			(mode 1)
-			(useauxorigin no)
+			(useauxorigin yes)
 			(hpglpennumber 1)
 			(hpglpenspeed 20)
@@
 			(pdf_single_document no)
 			(dxfpolygonmode yes)
-			(dxfimperialunits yes)
+			(dxfimperialunits no)
 			(dxfusepcbnewfont yes)
 			(psnegative no)
@@
 			(crossoutdnponfab yes)
 			(subtractmaskfromsilk no)
-			(outputformat 1)
+			(outputformat 3)
 			(mirror no)
-			(drillshape 0)
+			(drillshape 2)
 			(scaleselection 1)
-			(outputdirectory "gerber/")
+			(outputdirectory "dxf/")
 		)
 	)
@@
 		)
 	)
+	(footprint "Resistor_SMD:R_0805_2012Metric_Pad1.20x1.40mm_HandSolder"
+		(layer "F.Cu")
+		(at 167 89.2 180)
+		(descr "Resistor SMD 0805 (2012 Metric), square (rectangular) end terminal, IPC-7351 nominal with elongated pad for handsoldering. (Body size source: IPC-SM-782 page 72, https://www.pcb-3d.com/wordpress/wp-content/uploads/ipc-sm-782a_amendment_1_and_2.pdf), generated with kicad-footprint-generator")
+		(tags "resistor handsolder")
+		(property "Reference" "R4"
+			(at 0 -1.65 0)
+			(layer "F.SilkS")
+			(effects
+				(font
+					(size 1 1)
+					(thickness 0.15)
+				)
+			)
+		)
+		(property "Value" "10k"
+			(at 0 1.65 0)
+			(layer "F.Fab")
+			(effects
+				(font
+					(size 1 1)
+					(thickness 0.15)
+				)
+			)
+		)
+		(property "Datasheet" "~"
+			(at 0 0 0)
+			(layer "F.Fab")
+			(hide yes)
+			(effects
+				(font
+					(size 1.27 1.27)
+					(thickness 0.15)
+				)
+			)
+		)
+		(property "Description" "Resistor, small symbol"
+			(at 0 0 0)
+			(layer "F.Fab")
+			(hide yes)
+			(effects
+				(font
+					(size 1.27 1.27)
+					(thickness 0.15)
+				)
+			)
+		)
+		(property ki_fp_filters "R_*")
+		(sheetname "/")
+		(sheetfile "ColorMemo.kicad_sch")
+		(attr smd)
+		(fp_line
+			(start -0.227064 0.735)
+			(end 0.227064 0.735)
+			(stroke
+				(width 0.12)
+				(type solid)
+			)
+			(layer "F.SilkS")
+		)
+		(fp_line
+			(start -0.227064 -0.735)
+			(end 0.227064 -0.735)
+			(stroke
+				(width 0.12)
+				(type solid)
+			)
+			(layer "F.SilkS")
+		)
+		(fp_line
+			(start 1.85 0.95)
+			(end -1.85 0.95)
+			(stroke
+				(width 0.05)
+				(type solid)
+			)
+			(layer "F.CrtYd")
+		)
+		(fp_line
+			(start 1.85 -0.95)
+			(end 1.85 0.95)
+			(stroke
+				(width 0.05)
+				(type solid)
+			)
+			(layer "F.CrtYd")
+		)
+		(fp_line
+			(start -1.85 0.95)
+			(end -1.85 -0.95)
+			(stroke
+				(width 0.05)
+				(type solid)
+			)
+			(layer "F.CrtYd")
+		)
+		(fp_line
+			(start -1.85 -0.95)
+			(end 1.85 -0.95)
+			(stroke
+				(width 0.05)
+				(type solid)
+			)
+			(layer "F.CrtYd")
+		)
+		(fp_line
+			(start 1 0.625)
+			(end -1 0.625)
+			(stroke
+				(width 0.1)
+				(type solid)
+			)
+			(layer "F.Fab")
+		)
+		(fp_line
+			(start 1 -0.625)
+			(end 1 0.625)
+			(stroke
+				(width 0.1)
+				(type solid)
+			)
+			(layer "F.Fab")
+		)
+		(fp_line
+			(start -1 0.625)
+			(end -1 -0.625)
+			(stroke
+				(width 0.1)
+				(type solid)
+			)
+			(layer "F.Fab")
+		)
+		(fp_line
+			(start -1 -0.625)
+			(end 1 -0.625)
+			(stroke
+				(width 0.1)
+				(type solid)
+			)
+			(layer "F.Fab")
+		)
+		(fp_text user "${REFERENCE}"
+			(at 0 0 0)
+			(layer "F.Fab")
+			(effects
+				(font
+					(size 0.5 0.5)
+					(thickness 0.08)
+				)
+			)
+		)
+		(pad "1" smd roundrect
+			(at -1 0 180)
+			(size 1.2 1.4)
+			(layers "F.Cu" "F.Mask" "F.Paste")
+			(roundrect_rratio 0.208333)
+			(net 23 "VDD")
+			(pintype "passive")
+		)
+		(pad "2" smd roundrect
+			(at 1 0 180)
+			(size 1.2 1.4)
+			(layers "F.Cu" "F.Mask" "F.Paste")
+			(roundrect_rratio 0.208333)
+			(net 22 "/MUL_COL_3")
+			(pintype "passive")
+		)
+		(embedded_fonts no)
+		(model "${KICAD9_3DMODEL_DIR}/Resistor_SMD.3dshapes/R_0805_2012Metric.step"
+			(offset
+				(xyz 0 0 0)
+			)
+			(scale
+				(xyz 1 1 1)
+			)
+			(rotate
+				(xyz 0 0 0)
+			)
+		)
+	)
 	(footprint "Capacitor_SMD:C_0603_1608Metric"
 		(layer "F.Cu")
@@
 	)
 	(segment
+		(start 164.785 89.2)
+		(end 160.155 84.57)
+		(width 0.2)
+		(layer "F.Cu")
+		(net 22)
+	)
+	(segment
 		(start 158.604 100.331836)
 		(end 158.604 86.121)
@@
 	)
 	(segment
+		(start 166 89.2)
+		(end 164.785 89.2)
+		(width 0.2)
+		(layer "F.Cu")
+		(net 22)
+	)
+	(segment
 		(start 189.35 124.3)
 		(end 195.85 124.3)
@@
 	)
 	(segment
+		(start 164.4 87.6)
+		(end 164.4 78.655)
+		(width 0.2)
+		(layer "F.Cu")
+		(net 23)
+	)
+	(segment
+		(start 166.4 87.6)
+		(end 164.4 87.6)
+		(width 0.2)
+		(layer "F.Cu")
+		(net 23)
+	)
+	(segment
+		(start 168 89.2)
+		(end 166.4 87.6)
+		(width 0.2)
+		(layer "F.Cu")
+		(net 23)
+	)
+	(segment
+		(start 164.4 78.655)
+		(end 160.155 74.41)
+		(width 0.2)
+		(layer "F.Cu")
+		(net 23)
+	)
+	(segment
